File: BMS.kicad_sch (KiCad schematic)
At the start: 40 parts, among them J2 BMS1OTP, J3 BMS2OTP, U1 EL3H7, U2 BQ7695201PFBR, U3 ISO1640BDR, U5 BQ7695201PFBR, U6 ISO1640BDR

Commit message: BOOM
Parts:
- C11, C5: P/N (none) -> C0805C474K3RAC
- C12, C6: P/N (none) -> C0805C101FCGACTU
Changed lines of the file:
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@@
 			)
 		)
+		(property "P/N" "C0805C101FCGACTU"
+			(at 112.395 37.465 0)
+			(effects
+				(font
+					(size 1.27 1.27)
+				)
+				(hide yes)
+			)
+		)
 		(pin "1"
 		)
@@
 			)
 		)
+		(property "P/N" "C0805C474K3RAC"
+			(at 351.79 31.115 0)
+			(effects
+				(font
+					(size 1.27 1.27)
+				)
+				(hide yes)
+			)
+		)
 		(pin "1"
 		)
@@
 			)
 		)
+		(property "P/N" "C0805C101FCGACTU"
+			(at 365.76 32.385 0)
+			(effects
+				(font
+					(size 1.27 1.27)
+				)
+				(hide yes)
+			)
+		)
 		(pin "1"
 		)
@@
 			(at 98.425 36.195 0)
 			(effects
+				(font
+					(size 1.27 1.27)
+				)
+				(hide yes)
+			)
+		)
+		(property "P/N" "C0805C474K3RAC"
+			(at 98.425 36.195 0)
+			(effects
