File: BPS-Minion.kicad_pcb (KiCad board)
At the start: 2 copper layers, 160 x 63 mm, 226 parts, among them J1 TEMPSPIANALYZER, J10 TopConn, J11 TopConn, J12 TEMPSPIANALYZER, J13 CAN_IN, J14 CAN_OUT, J2 BMS1OTP, J3 BMS2OTP, J4 Conn_01x24_Female, J5 Conn_01x24_Female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

Commit message: BOOM
Routing:
- net /SPI1_MISO: track 39.2 -> 65.6 mm
- net /SPI1_SCK: track 45.2 -> 67.3 mm
- net GNDA: track 55.2 -> 54.6 mm
Other:
- board text added: "GND"
- board text added: "MISO"
- board text added: "MOSI"
- board text added: "SCL"
- board text added: "SDA"
- board text added: "sck"
