File: BatteryConnector.kicad_sch (KiCad schematic)
At the start: 19 parts, among them J6 TopConn

Commit message: BOOM
Parts:
- C25, C26, C27, C28, C29, C30: P/N (none) -> C0805C224K5RACTU
- R53, R54, R55, R56, R57, R58: P/N (none) -> RCS080520R0FKEA
Changed lines of the file:
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@@
+			)
+		)
+		(property "P/N" "RCS080520R0FKEA"
+			(at 98.425 75.565 0)
+			(effects
+				(font
+					(size 1.27 1.27)
+				)
+				(hide yes)
 			)
 		)
@@
 			)
 		)
+		(property "P/N" "C0805C224K5RACTU"
+			(at 133.985 88.265 0)
+			(effects
+				(font
+					(size 1.27 1.27)
+				)
+				(hide yes)
+			)
+		)
 		(pin "1"
 		)
@@
 			)
 		)
+		(property "P/N" "RCS080520R0FKEA"
+			(at 118.745 75.565 0)
+			(effects
+				(font
+					(size 1.27 1.27)
+				)
+				(hide yes)
+			)
+		)
 		(pin "1"
 		)
@@
 			)
 		)
+		(property "P/N" "C0805C224K5RACTU"
+			(at 113.665 88.265 0)
+			(effects
+				(font
+					(size 1.27 1.27)
+				)
+				(hide yes)
+			)
+		)
 		(pin "1"
 		)
@@
 			)
 		)
+		(property "P/N" "RCS080520R0FKEA"
+			(at 108.585 75.565 0)
+			(effects
+				(font
+					(size 1.27 1.27)
+				)
+				(hide yes)
+			)
+		)
 		(pin "1"
 		)
@@
 			)
 		)
+		(property "P/N" "C0805C224K5RACTU"
+			(at 83.185 88.265 0)
+			(effects
+				(font
+					(size 1.27 1.27)
+				)
+				(hide yes)
+			)
+		)
 		(pin "1"
 		)
@@
 			)
 		)
+		(property "P/N" "RCS080520R0FKEA"
+			(at 88.265 75.565 0)
+			(effects
+				(font
+					(size 1.27 1.27)
+				)
+				(hide yes)
+			)
+		)
 		(pin "1"
 		)
@@
 			)
 		)
+		(property "P/N" "C0805C224K5RACTU"
+			(at 103.505 88.265 0)
+			(effects
+				(font
+					(size 1.27 1.27)
+				)
+				(hide yes)
+			)
+		)
 		(pin "1"
 		)
@@
 			)
 		)
+		(property "P/N" "RCS080520R0FKEA"
+			(at 139.065 75.565 0)
+			(effects
+				(font
+					(size 1.27 1.27)
+				)
+				(hide yes)
+			)
+		)
 		(pin "1"
 		)
@@
 			)
 		)
+		(property "P/N" "C0805C224K5RACTU"
+			(at 93.345 88.265 0)
+			(effects
+				(font
+					(size 1.27 1.27)
+				)
+				(hide yes)
+			)
+		)
 		(pin "1"
 		)
@@
 			)
 		)
+		(property "P/N" "RCS080520R0FKEA"
+			(at 128.905 75.565 0)
+			(effects
+				(font
+					(size 1.27 1.27)
+				)
+				(hide yes)
+			)
+		)
 		(pin "1"
 		)
@@
 			(at 123.825 88.265 0)
 			(effects
+				(font
+					(size 1.27 1.27)
+				)
+				(hide yes)
+			)
+		)
+		(property "P/N" "C0805C224K5RACTU"
+			(at 123.825 88.265 0)
+			(effects
