File: Temperature.kicad_sch (KiCad schematic)
At the start: 30 parts, among them J1 TEMPSPIANALYZER, J3 Conn_01x24_Female, U8 LM321, U9 ADS7953SBDBT

Commit message: BOOM
Parts:
- C16, C17: P/N (none) -> KAM21BR71H473KT
Changed lines of the file:
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@@
 			)
 		)
+		(property "P/N" "KAM21BR71H473KT"
+			(at 195.58 104.775 0)
+			(effects
+				(font
+					(size 1.27 1.27)
+				)
+				(hide yes)
+			)
+		)
 		(pin "1"
 		)
@@
 			(at 213.36 104.775 0)
 			(effects
+				(font
+					(size 1.27 1.27)
+				)
+				(hide yes)
+			)
+		)
+		(property "P/N" "KAM21BR71H473KT"
+			(at 213.36 104.775 0)
+			(effects

Commit message: grrrrr
Parts:
- U8: P/N LM321 -> LM321MF/NOPB
Changed lines of the file:
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@@
 			)
 		)
-		(property "P/N" "LM321"
+		(property "P/N" "LM321MF/NOPB "
 			(at 232.41 103.505 0)
 			(effects
